File: Docs/KiCad/DomoticShutterPanel.kicad_pcb (KiCad board)
At the start: 2 copper layers, 107.1 x 48 mm, 24 parts, among them J1 Conn_01x12, J2 Conn_01x02, J3 Conn_01x06, J4 Conn_01x02, J5 Conn_01x12, K1 SRD-05VDC-SL-C

Commit message: Changed to radio approach
Parts:
- removed J1, J5: Conn_01x12, Socket_Arduino_Pro_Mini:Socket_Strip_Arduino_1x12
- removed J2, J4: Conn_01x02, Socket_Arduino_Pro_Mini:Socket_Strip_Arduino_1x02
- removed J3: Conn_01x06, Socket_Arduino_Pro_Mini:Socket_Strip_Arduino_1x06
- removed K1 (x7): SRD-05VDC-SL-C, Custom_libraries:RELAY_SRD-05VDC-SL-C
- removed the REF** at (199.0, 114.0)
- removed the REF** at (139.0, 115.0)
- removed the REF** at (200.0, 114.0)
- removed the REF** at (137.0, 132.0)
- removed the REF** at (192.0, 80.0)
- removed the REF** at (175.0, 80.0)
- removed the REF** at (158.0, 80.0)
- removed the REF** at (141.0, 80.0)
- removed the REF** at (124.0, 80.0)
- removed the REF** at (107.0, 80.0)
- removed the REF** at (102.0, 115.0)
Other:
- board outline removed
- board text removed: "DTR"
- board text removed: "GND"
- board text removed: "RX1"
- board text removed: "TX0"
