File: Docs/KiCad/DomoticShutterPanel.sch (KiCad schematic (older format))
At the start: 37 parts, among them J1 Conn_01x02, J2 3.3V DC-DC Step-Down Power Mo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, J3 Conn_01x04, J4 BOOT OPTION, J5 UART COM, J9 Conn_01x03, SW1 SW_Push, SW2 SW_Push, SW3 SW_Push, SW4 SW_Push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

Commit message: Schematic cleanup and new 3d models
3d models for S8550 and PS2701
Parts:
- removed C1, C2, C3, C4, C?: 1uF, Capacitor_THT:C_Radial_D5.0mm_H5.0mm_P2.00mm, symbol CustomLibraries_Device:CP
- removed C5, C6: 0.1uF, Capacitor_THT:C_Radial_D5.0mm_H5.0mm_P2.00mm, symbol CustomLibraries_Device:C
- removed C?: 10uF, symbol CustomLibraries_Device:C
- removed J1: Conn_01x02, Custom_libraries:PinSocket_1x02_P2.54mm_Vertical, symbol CustomLibraries_connectors:Conn_01x02
- removed J2: 3.3V DC-DC Step-Down Power Module, Custom_libraries:DCDC_3v3_PowerModule, symbol CustomLibraries_connectors:Conn_02x02_Odd_Even
- removed J4: BOOT OPTION, Connector_PinHeader_2.54mm:PinHeader_1x02_P2.54mm_Vertical, symbol CustomLibraries_connectors:Conn_01x02
- removed J9: Conn_01x03, Connector_PinHeader_2.54mm:PinHeader_1x03_P2.54mm_Vertical, symbol CustomLibraries_connectors:Conn_01x03
- removed R1, R2, R3, R4, R?: 15k, Resistor_THT:R_Axial_DIN0204_L3.6mm_D1.6mm_P1.90mm_Vertical, symbol CustomLibraries_Device:R
- removed R8, R9: 10k, Resistor_THT:R_Axial_DIN0204_L3.6mm_D1.6mm_P1.90mm_Vertical, symbol CustomLibraries_Device:R
- removed SW1, SW2, SW3, SW4, SW5, SW?: SW_Push, Custom_libraries:SW_PUSH_6mm, symbol CustomLibraries_Switch:SW_Push
- added C? (x2): 0.1uF, symbol CustomLibraries_Device:C
- added C?: 47uF, symbol CustomLibraries_Device:CP
- added C? (x2): 0.1uF, Capacitor_THT:C_Radial_D5.0mm_H5.0mm_P2.00mm, symbol CustomLibraries_Device:C
- added C?: 10uF, symbol CustomLibraries_Device:CP
- added C? (x5): 1uF, Capacitor_THT:C_Radial_D5.0mm_H5.0mm_P2.00mm, symbol CustomLibraries_Device:C
- added D?: 1N4007, symbol CustomLibraries_Device:D
- added D?: LED, symbol CustomLibraries_Device:LED
- added D?: LED1, symbol CustomLibraries_Device:LED
- added J?: PWR 5V AUX, symbol Connector:USB_B_Mini
- added J?: PWR SEL, Connector_PinHeader_2.54mm:PinHeader_1x03_P2.54mm_Vertical, symbol CustomLibraries_connectors:Conn_01x03
- added J?: PWR 5V, symbol Connector:Screw_Terminal_01x02
- added J?: SLAVE UART COM, Connector_PinHeader_2.54mm:PinHeader_1x04_P2.54mm_Vertical, symbol CustomLibraries_connectors:Conn_01x04
- added J?: TRIGGER SEL, Connector_PinHeader_2.54mm:PinHeader_1x03_P2.54mm_Vertical, symbol CustomLibraries_connectors:Conn_01x03
- added J?: Screw_Terminal_01x03, symbol Connector:Screw_Terminal_01x03
- added K?: SRD-05VDC-SL-C, RELAY_SRD-05VDC-SL-C, symbol CustomLibraries_SRD-05VDC-SL-C:SRD-05VDC-SL-C
- added Q?: S8550, Package_TO_SOT_SMD:SOT-23, symbol CustomLibraries_Device:S8550
- added R? (x2): 1k, symbol CustomLibraries_Device:R
- added R?: 2.2k, symbol CustomLibraries_Device:R
- added R?: 10k, symbol CustomLibraries_Device:R
- added R?: 15k, symbol CustomLibraries_Device:R
- added R? (x2): 10k, Resistor_THT:R_Axial_DIN0204_L3.6mm_D1.6mm_P1.90mm_Vertical, symbol CustomLibraries_Device:R
- added R? (x5): 15k, Resistor_THT:R_Axial_DIN0204_L3.6mm_D1.6mm_P1.90mm_Vertical, symbol CustomLibraries_Device:R
- added SW?: BOOT, Custom_libraries:SW_PUSH_6mm, symbol CustomLibraries_Switch:SW_Push
- added SW?: RESET, Custom_libraries:SW_PUSH_6mm, symbol CustomLibraries_Switch:SW_Push
- added SW? (x4): SW_Push, Custom_libraries:SW_PUSH_6mm, symbol CustomLibraries_Switch:SW_Push
- added SW?: LAMP, Custom_libraries:SW_PUSH_6mm, symbol CustomLibraries_Switch:SW_Push
- added U?: 3v3 DCDC Converter Power Module, symbol Project_Library:3v3_DCDC_Converter_Power_Module
- added U?: PS2705-1, symbol CustomLibraries_Device:PS2705-1
- J?: renamed from J3; value Conn_01x04 -> LCD COM
- J?: value RF_Rx -> RF RX
- J?: value RF_Tx -> RF TX
- J?: renamed from J5; value UART COM -> MASTER UART COM
- U2: value Arduino_MiniPro -> Shield Arduino Pro Mini 3v3; footprint Custom_libraries:Socket_Strip_Arduino_MiniPro -> Custom_libraries:Socket_Strip_Arduino_MiniPro_3V3; symbol CustomLibraries_connectors:Arduino_MiniPro -> Project_Library:Arduino_ProMini_3V3
- renumbered R7 to R?, R5 to R?
Connections:
- net labels added: U1_GPIO0, U1_RST
- net labels removed: +3.3V, 10, 11, 12, 13, 4, 6, 8, 9, A0, A1, A2, A3, A6, A7, RAW, Reset
- wire segments 186 -> 162
- no-connect marks 14 -> 23
Other:
- note added: "AUDIO"
- note added: "BUTTONS"
- note added: "COMMUNICATION HEADERS"
- note added: "I2C RESISTORS"
- note added: "MASTER"
- note added: "MICROCONTROLLERS"
- note added: "POWER"
- note added: "RELAY"
- note added: "SLAVE"
- note removed: "1"
- note removed: "3.3V DC-DC Step-Down \nPower Module"
- note removed: "Button setup"
- note removed: "Buzzer"
- note removed: "ESP-WROOM-02"
- note removed: "I2C PULLUP RESISTOR"
- note removed: "LCD 16x2 I2C"
- note removed: "Lamp Relay"
- note removed: "Lamp button"
- note removed: "Radio modules"
- note removed: "Shield Arduino Pro Mini \n"
- moved on the sheet: C?, J?, LS?, R?, U1

Commit message: Unified libraries to one
Parts:
- added D1: 1N5822, Diode_THT:D_DO-201AD_P15.24mm_Horizontal, symbol Diode:1N5822
- C1, C4: renamed from C?; symbol CustomLibraries_Device:CP -> Device:CP
- C10, C11, C12, C2, C3, C5, C6, C7, C8, C9: renamed from C?; symbol CustomLibraries_Device:C -> Device:C
- D2, D4: renamed from D?; symbol CustomLibraries_Device:LED -> Device:LED
- D3: renamed from D?; symbol CustomLibraries_Device:D -> Device:D
- J10, J7, J9: renamed from J?; symbol CustomLibraries_connectors:Conn_01x04 -> Connector_Generic:Conn_01x04
- J3, J4, J6, J8: renamed from J?; symbol CustomLibraries_connectors:Conn_01x03 -> Connector_Generic:Conn_01x03
- K1: renamed from K?; symbol CustomLibraries_SRD-05VDC-SL-C:SRD-05VDC-SL-C -> Project_Library:SRD-05VDC-SL-C
- LS1: renamed from LS?; symbol CustomLibraries_Device:Speaker -> Device:Speaker
- Q1: renamed from Q?; symbol CustomLibraries_Device:S8550 -> Project_Library:S8550
- R1, R10, R11, R12, R13, R14, R15, R16, R2, R3, R4, R5, R6, R7, R8, R9: renamed from R?; symbol CustomLibraries_Device:R -> Device:R
- SW1, SW2, SW3, SW4, SW5, SW6, SW7: renamed from SW?; symbol CustomLibraries_Switch:SW_Push -> Switch:SW_Push
- U1: renamed from U?; symbol CustomLibraries_Device:PS2705-1 -> Project_Library:PS2705-1
- U3: renamed from U1; symbol ESP8266:ESP-13-WROOM-02 -> Project_Library:ESP-13-WROOM-02
- gave numbers to parts that had none: 4
- renumbered U2 to U4
Connections:
- net DATA_Tx: now also U4.12 (D9)
- net at J4.1 (Pin_1): now also D1.1 (K); no longer J1.1 (Pin_1)
- new net: D1.2 (A), J1.1 (Pin_1)
- no-connect marks 23 -> 22
Other:
- moved on the sheet: J1
