File: PCB_Design/DomoticShutterPanel.kicad_pcb (KiCad board)
At the start: 2 copper layers, 110.6 x 50 mm, 62 parts, among them J1 PWR 5V, J10 LCD COM, J2 PWR 5V AUX, J3 TRIGGER SEL, J4 PWR SEL, J5 Screw_Terminal_01x03, J6 RF TX, J7 RF RX, J8 MASTER UART COM, J9 LAMP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

Commit message: Ready to production
Parts:
- added G***: LOGO, Project_libraries:MickySim_Logo_6mm, F.Cu at (183.3, 120.8)
- added REF**: OSHW-Logo2_7.3x6mm_SilkScreen, Symbol:OSHW-Logo2_7.3x6mm_SilkScreen, B.Cu at (196.5, 120.8)
- added REF**: KiCad-Logo_5mm_SilkScreen, Symbol:KiCad-Logo_5mm_SilkScreen, B.Cu at (185.5, 120.8)
- moved D1 3.57 mm to (114.7, 120.5)
Routing:
- net Net-(D1-Pad1): track 10.8 -> 5.79 mm
- net +3V3: track 165.3 -> 162.4 mm
- net +5V: track 168.8 -> 171.1 mm
- net Net-(D1-Pad2): track 8.12 -> 9.76 mm
Other:
- net class Default: clearance 0.1778 -> 0.2032
- rule trace_clearance: 0.1778 -> 0.2032
- board text added: "5V"
- board text added: "ANALOG"
- board text added: "CAUTION 230 VAC"
- board text added: "DIGITAL"
- board text added: "HIGH"
- board text added: "I2C RESISTORS"
- board text added: "KEEP-OUT"
- board text added: "LOW"
- board text added: "NO COPPER AREA"
- board text added: "ON ALL LAYER"
- board text added: "PWR_5V"
- board text added: "PWR_USB"
- board text added: "ROLLER SHUTTER CONTROL BOARD"
- board text added: "RX"
- board text added: "Rev 1.0"
- board text added: "SCL"
- board text added: "SDA"
- board text added: "THIS SIDE BOTTOM"
- board text added: "THIS SIDE UP"
- board text added: "TX"
