File: PCB_Design/DomoticShutterPanel.sch (KiCad schematic (older format))
At the start: 56 parts, among them J1 PWR 5V, J10 LCD COM, J2 PWR 5V AUX, J3 TRIGGER SEL, J4 PWR SEL, J5 Screw_Terminal_01x03, J6 RF TX, J7 RF RX, J8 MASTER UART COM, J9 SLAVE UART COM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

Commit message: Updated 3D models and schematic
Arduino symbol changed in schematic. The UART connector is no longer displayed and I can be accessed externaly.
New 3D models for 400mhz modules, buzzer and conectors.
Parts:
- removed J9: SLAVE UART COM, Connector_PinHeader_2.54mm:PinHeader_1x04_P2.54mm_Vertical, symbol Connector_Generic:Conn_01x04
- C1, C4: footprint (none) -> Capacitor_THT:CP_Radial_D4.0mm_P2.00mm
- C10, C11, C12, C6, C7, C8, C9: footprint Capacitor_THT:C_Radial_D5.0mm_H5.0mm_P2.00mm -> Capacitor_SMD:C_1206_3216Metric_Pad1.42x1.75mm_HandSolder
- C2, C3, C5: footprint (none) -> Capacitor_SMD:C_1206_3216Metric_Pad1.42x1.75mm_HandSolder
- D1: footprint Diode_THT:D_DO-201AD_P15.24mm_Horizontal -> Diode_THT:D_DO-201AD_P5.08mm_Vertical_KathodeUp
- D2, D4: footprint (none) -> LED_THT:LED_D3.0mm
- D3: footprint (none) -> Diode_THT:D_DO-41_SOD81_P10.16mm_Horizontal
- J1: footprint (none) -> Project_libraries:PHOENIX_1935161
- J10, J7: footprint Connector_PinHeader_2.54mm:PinHeader_1x04_P2.54mm_Vertical -> Connector_PinSocket_2.54mm:PinSocket_1x04_P2.54mm_Vertical
- J2: footprint (none) -> Connector_USB:USB_Mini-B_Lumberg_2486_01_Horizontal
- J5: footprint (none) -> Project_libraries:ScrewTerminal_01X03_5mm
- J6: footprint Connector_PinHeader_2.54mm:PinHeader_1x03_P2.54mm_Vertical -> Connector_PinSocket_2.54mm:PinSocket_1x03_P2.54mm_Vertical
- K1: footprint RELAY_SRD-05VDC-SL-C -> Project_libraries:RELAY_SRD-05VDC-SL-C
- LS1: footprint (none) -> Buzzer_Beeper:Buzzer_TDK_PS1240P02BT_D12.2mm_H6.5mm
- Q1: footprint Package_TO_SOT_SMD:SOT-23 -> Project_libraries:SOT-23_S8550
- R1, R2, R3, R4, R7, R8, R9: footprint (none) -> Resistor_THT:R_Axial_DIN0204_L3.6mm_D1.6mm_P5.08mm_Horizontal
- R10, R11, R12, R13, R14, R15, R16, R5, R6: footprint Resistor_THT:R_Axial_DIN0204_L3.6mm_D1.6mm_P1.90mm_Vertical -> Resistor_THT:R_Axial_DIN0204_L3.6mm_D1.6mm_P5.08mm_Horizontal
- SW1, SW2, SW3, SW4, SW5, SW6: footprint Custom_libraries:SW_PUSH_6mm -> Project_libraries:SW_PUSH_6mm
- SW7: footprint Custom_libraries:SW_PUSH_6mm -> Project_libraries:PHOENIX_1935161
- U1: footprint (none) -> Project_libraries:PS2705-1-F3
- U2: footprint (none) -> Project_libraries:DCDC_3v3_PowerModule
- U3: footprint Custom_libraries:ESP-13-WROOM-02 -> Project_libraries:ESP-13-WROOM-02
- U4: footprint Custom_libraries:Socket_Strip_Arduino_MiniPro_3V3 -> Project_libraries:Socket_Strip_Arduino_MiniPro
Connections:
- net +5V: now also J7.4 (Pin_4); no longer J7.1 (Pin_1)
- net GND: now also J7.1 (Pin_1); no longer J7.4 (Pin_4)
- net PWR_USB: now reaches J2.1 (VBUS), J4.3 (Pin_3)
Other:
- moved on the sheet: J10

Commit message: Changed to SMD pushbutton
Parts:
- SW1, SW2, SW3, SW4, SW5, SW6: footprint Project_libraries:SW_PUSH_6mm -> Project_libraries:SW_Push_1P1T_NO_6x6mm_H5mm
Changed lines of the file:
@@
 F 0 "SW4" V 7750 1500 50  0000 L CNN
 F 1 "SW_Push" V 7650 1550 50  0000 C CNN
-F 2 "Project_libraries:SW_PUSH_6mm" H 7700 1950 50  0001 C CNN
+F 2 "Project_libraries:SW_Push_1P1T_NO_6x6mm_H5mm" H 7700 1950 50  0001 C CNN
 F 3 "~" H 7700 1950 50  0001 C CNN
 	1    7700 1750
@@
 F 0 "SW3" V 6800 1500 50  0000 L CNN
 F 1 "SW_Push" V 6700 1550 50  0000 C CNN
-F 2 "Project_libraries:SW_PUSH_6mm" H 6750 1950 50  0001 C CNN
+F 2 "Project_libraries:SW_Push_1P1T_NO_6x6mm_H5mm" H 6750 1950 50  0001 C CNN
 F 3 "~" H 6750 1950 50  0001 C CNN
 	1    6750 1750
@@
 F 0 "SW2" V 5850 1500 50  0000 L CNN
 F 1 "SW_Push" V 5750 1550 50  0000 C CNN
-F 2 "Project_libraries:SW_PUSH_6mm" H 5800 1950 50  0001 C CNN
+F 2 "Project_libraries:SW_Push_1P1T_NO_6x6mm_H5mm" H 5800 1950 50  0001 C CNN
 F 3 "~" H 5800 1950 50  0001 C CNN
 	1    5800 1750
@@
 F 0 "SW1" V 4900 1500 50  0000 L CNN
 F 1 "SW_Push" V 4800 1550 50  0000 C CNN
-F 2 "Project_libraries:SW_PUSH_6mm" H 4850 1950 50  0001 C CNN
+F 2 "Project_libraries:SW_Push_1P1T_NO_6x6mm_H5mm" H 4850 1950 50  0001 C CNN
 F 3 "~" H 4850 1950 50  0001 C CNN
 	1    4850 1750
@@
 F 0 "SW6" V 9750 1500 50  0000 L CNN
 F 1 "RESET" V 9650 1450 50  0000 L CNN
-F 2 "Project_libraries:SW_PUSH_6mm" H 9700 1950 50  0001 C CNN
+F 2 "Project_libraries:SW_Push_1P1T_NO_6x6mm_H5mm" H 9700 1950 50  0001 C CNN
 F 3 "~" H 9700 1950 50  0001 C CNN
 	1    9700 1750
@@
 F 0 "SW5" V 8800 1500 50  0000 L CNN
 F 1 "BOOT" V 8700 1600 50  0000 C CNN
-F 2 "Project_libraries:SW_PUSH_6mm" H 8750 1950 50  0001 C CNN
+F 2 "Project_libraries:SW_Push_1P1T_NO_6x6mm_H5mm" H 8750 1950 50  0001 C CNN
 F 3 "~" H 8750 1950 50  0001 C CNN
 	1    8750 1750

Commit message: R and C added for buttons
Parts:
- J8: footprint Connector_PinHeader_2.54mm:PinHeader_1x03_P2.54mm_Vertical -> Connector_PinHeader_2.54mm:PinHeader_1x04_P2.54mm_Vertical; symbol Connector_Generic:Conn_01x03 -> Connector_Generic:Conn_01x04
Connections:
- net +3V3: now also J8.2 (Pin_2)
- net U1_RXD: now also J8.4 (Pin_4); no longer J8.3 (Pin_3)
- net U1_TXD: now also J8.3 (Pin_3); no longer J8.2 (Pin_2)
Other:
- moved on the sheet: J10
Changed lines of the file:
@@
 EESchema Schematic File Version 4
-LIBS:DomoticShutterPanel-cache
-EELAYER 29 0
+EELAYER 30 0
 EELAYER END
 $Descr A4 11693 8268
@@
 	650  2550 8400 2550
 $Comp
-L Connector_Generic:Conn_01x03 J8
+L Connector_Generic:Conn_01x04 J8
 U 1 1 5EA8DAF9
 P 10050 4450
 F 0 "J8" H 10130 4492 50  0000 L CNN
 F 1 "MASTER UART COM" H 10130 4401 50  0000 L CNN
-F 2 "Connector_PinHeader_2.54mm:PinHeader_1x03_P2.54mm_Vertical" H 10050 4450 50  0001 C CNN
+F 2 "Connector_PinHeader_2.54mm:PinHeader_1x04_P2.54mm_Vertical" H 10050 4450 50  0001 C CNN
 F 3 "~" H 10050 4450 50  0001 C CNN
 	1    10050 4450
@@
 	9800 3850 9450 3850
 Wire Wire Line
-	9850 4550 9450 4550
-Wire Wire Line
-	9850 4450 9450 4450
+	9850 4650 9450 4650
+Text GLabel 9450 4650 0    39   Input ~ 0
+U1_RXD
 Text GLabel 9450 4550 0    39   Input ~ 0
-U1_RXD
-Text GLabel 9450 4450 0    39   Input ~ 0
 U1_TXD
 Text GLabel 9450 3850 0    39   Input ~ 0
@@
 	9550 3350 9550 3150
 Wire Wire Line
-	9850 5150 9450 5150
-Wire Wire Line
-	9450 5050 9850 5050
+	9850 5250 9450 5250
+Wire Wire Line
+	9450 5150 9850 5150
+Text GLabel 9450 5250 0    39   Input ~ 0
+I2C_SCL
 Text GLabel 9450 5150 0    39   Input ~ 0
-I2C_SCL
-Text GLabel 9450 5050 0    39   Input ~ 0
 I2C_SDA
 Wire Wire Line
-	9550 4950 9850 4950
-Wire Wire Line
-	9700 4850 9700 5350
-Wire Wire Line
-	9850 4850 9700 4850
+	9550 5050 9850 5050
+Wire Wire Line
+	9700 4950 9700 5450
+Wire Wire Line
+	9850 4950 9700 4950
 $Comp
 L power:GND #PWR050
 U 1 1 5F64D813
-P 9700 5350
-F 0 "#PWR050" H 9700 5100 50  0001 C CNN
-F 1 "GND" H 9700 5200 50  0000 C CNN
-F 2 "" H 9700 5350 50  0001 C CNN
-F 3 "" H 9700 5350 50  0001 C CNN
-	1    9700 5350
+P 9700 5450
+F 0 "#PWR050" H 9700 5200 50  0001 C CNN
+F 1 "GND" H 9700 5300 50  0000 C CNN
+F 2 "" H 9700 5450 50  0001 C CNN
+F 3 "" H 9700 5450 50  0001 C CNN
+	1    9700 5450
 	1    0    0    -1
 $EndComp
@@
 L Connector_Generic:Conn_01x04 J10
 U 1 1 5EA32128
-P 10050 4950
-F 0 "J10" H 10130 4942 50  0000 L CNN
-F 1 "LCD COM" H 10130 4851 50  0000 L CNN
-F 2 "Connector_PinSocket_2.54mm:PinSocket_1x04_P2.54mm_Vertical" H 10050 4950 50  0001 C CNN
-F 3 "~" H 10050 4950 50  0001 C CNN
-	1    10050 4950
-	1    0    0    -1
-$EndComp
-Wire Wire Line
-	9700 4850 9700 4350
-Connection ~ 9700 4850
-Connection ~ 9700 4350
+P 10050 5050
+F 0 "J10" H 10130 5042 50  0000 L CNN
+F 1 "LCD COM" H 10130 4951 50  0000 L CNN
+F 2 "Connector_PinSocket_2.54mm:PinSocket_1x04_P2.54mm_Vertical" H 10050 5050 50  0001 C CNN
+F 3 "~" H 10050 5050 50  0001 C CNN
+	1    10050 5050
+	1    0    0    -1
+$EndComp
 Wire Notes Line
 	8850 2550 8850 5700
@@
 Wire Wire Line
 	9850 4050 9550 4050
+Wire Wire Line
+	9450 4550 9850 4550
+Wire Wire Line
+	9550 4050 9550 5050
 Connection ~ 9550 4050
 Wire Wire Line
-	9550 4050 9550 4950
+	9850 4450 9400 4450
+Wire Wire Line
+	9400 4450 9400 4350
+$Comp
+L power:+3V3 #PWR?
+U 1 1 5F7382DD
+P 9400 4350
+F 0 "#PWR?" H 9400 4200 50  0001 C CNN
+F 1 "+3V3" H 9415 4523 50  0000 C CNN
+F 2 "" H 9400 4350 50  0001 C CNN
+F 3 "" H 9400 4350 50  0001 C CNN
+	1    9400 4350
+	1    0    0    -1
+$EndComp
+Wire Wire Line
+	9700 4350 9700 4950
+Connection ~ 9700 4350
+Connection ~ 9700 4950
 $EndSCHEMATC

Commit message: Positioned all footprints
Parts:
- J9: renamed from SW7; symbol Switch:SW_Push -> Connector:Screw_Terminal_01x02
Connections:
- net GND: now also J1.1 (Pin_1); no longer J1.2 (Pin_2)
- net at D1.2 (A): now also J1.2 (Pin_2); no longer J1.1 (Pin_1)
Changed lines of the file:
@@
 Wire Notes Line
 	11000 2300 11000 750
-$Comp
-L Connector:Screw_Terminal_01x02 J1
-U 1 1 5F6B3CD7
-P 900 1000
-F 0 "J1" H 900 1250 50  0000 C CNN
-F 1 "PWR 5V" H 900 1150 50  0000 C CNN
-F 2 "Project_libraries:PHOENIX_1935161" H 900 1000 50  0001 C CNN
-F 3 "~" H 900 1000 50  0001 C CNN
-	1    900  1000
-	-1   0    0    -1
-$EndComp
 Text Notes 3500 750  0    79   ~ 0
 POWER
@@
 Wire Wire Line
 	10350 1600 10350 1500
-Wire Wire Line
-	10650 1550 10650 1500
 $Comp
 L Device:R R16
@@
 $EndComp
 $Comp
-L Switch:SW_Push SW7
+L Connector:Screw_Terminal_01x02 J9
 U 1 1 5FE3CC4F
-P 10650 1750
-F 0 "SW7" V 10700 1500 50  0000 L CNN
-F 1 "LAMP" V 10600 1500 50  0000 L CNN
-F 2 "Project_libraries:PHOENIX_1935161" H 10650 1950 50  0001 C CNN
-F 3 "~" H 10650 1950 50  0001 C CNN
-	1    10650 1750
-	0    -1   -1   0
+P 10850 1800
+F 0 "J9" H 10800 1500 50  0000 L CNN
+F 1 "LAMP" H 10750 1600 50  0000 L CNN
+F 2 "Project_libraries:PHOENIX_1935161" H 10850 2000 50  0001 C CNN
+F 3 "~" H 10850 2000 50  0001 C CNN
+	1    10850 1800
+	1    0    0    1
 $EndComp
 $Comp
@@
 $EndComp
 $Comp
-L Switch:SW_Push SW6
-U 1 1 5FD62E8D
-P 9700 1750
-F 0 "SW6" V 9750 1500 50  0000 L CNN
-F 1 "RESET" V 9650 1450 50  0000 L CNN
-F 2 "Project_libraries:SW_Push_1P1T_NO_6x6mm_H5mm" H 9700 1950 50  0001 C CNN
-F 3 "~" H 9700 1950 50  0001 C CNN
-	1    9700 1750
-	0    -1   -1   0
-$EndComp
-$Comp
-L Device:C C10
-U 1 1 5F64C379
-P 8450 1750
-F 0 "C10" H 8700 1700 50  0000 R CNN
-F 1 "0.1uF" H 8750 1800 50  0000 R CNN
-F 2 "Capacitor_SMD:C_1206_3216Metric_Pad1.42x1.75mm_HandSolder" H 8488 1600 50  0001 C CNN
-F 3 "~" H 8450 1750 50  0001 C CNN
-	1    8450 1750
-	-1   0    0    1
-$EndComp
-Wire Wire Line
-	8750 2000 8750 1950
-Wire Wire Line
-	8750 1950 8450 1950
-Wire Wire Line
-	8450 1950 8450 1900
-Wire Wire Line
-	8750 1500 8750 1450
-Connection ~ 8750 1500
-Wire Wire Line
-	8450 1500 8750 1500
-Wire Wire Line
-	8450 1600 8450 1500
-Wire Wire Line
-	8750 1550 8750 1500
-$Comp
-L Device:R R14
-U 1 1 5EB2F921
-P 8750 1300
-F 0 "R14" H 8900 1250 50  0000 C CNN
-F 1 "10k" H 8900 1350 50  0000 C CNN
-F 2 "Resistor_THT:R_Axial_DIN0204_L3.6mm_D1.6mm_P5.08mm_Horizontal" V 8680 1300 50  0001 C CNN
-F 3 "~" H 8750 1300 50  0001 C CNN
-	1    8750 1300
-	-1   0    0    1
-$EndComp
-$Comp
-L power:+3V3 #PWR045
-U 1 1 5EB09053
-P 8750 1150
-F 0 "#PWR045" H 8750 1000 50  0001 C CNN
-F 1 "+3V3" H 8750 1300 50  0000 C CNN
-F 2 "" H 8750 1150 50  0001 C CNN
-F 3 "" H 8750 1150 50  0001 C CNN
-	1    8750 1150
-	1    0    0    -1
-$EndComp
-$Comp
-L power:GND #PWR046
-U 1 1 5EAF6562
-P 8750 2000
-F 0 "#PWR046" H 8750 1750 50  0001 C CNN
-F 1 "GND" H 8755 1827 50  0000 C CNN
-F 2 "" H 8750 2000 50  0001 C CNN
-F 3 "" H 8750 2000 50  0001 C CNN
-	1    8750 2000
-	1    0    0    -1
-$EndComp
-$Comp
-L Switch:SW_Push SW5
-U 1 1 5F641C24
-P 8750 1750
-F 0 "SW5" V 8800 1500 50  0000 L CNN
-F 1 "BOOT" V 8700 1600 50  0000 C CNN
-F 2 "Project_libraries:SW_Push_1P1T_NO_6x6mm_H5mm" H 8750 1950 50  0001 C CNN
-F 3 "~" H 8750 1950 50  0001 C CNN
-	1    8750 1750
-	0    -1   -1   0
-$EndComp
-$Comp
 L power:GND #PWR032
 U 1 1 5FC9273E
@@
 Text GLabel 7400 1500 0    39   Input ~ 0
 U1_GPIO13
-Text GLabel 8450 1500 0    39   Input ~ 0
-U1_GPIO0
 Text GLabel 9400 1500 0    39   Input ~ 0
 U1_RST
@@
 	9400 4450 9400 4350
 $Comp
-L power:+3V3 #PWR?
+L power:+3V3 #PWR0103
 U 1 1 5F7382DD
 P 9400 4350
-F 0 "#PWR?" H 9400 4200 50  0001 C CNN
+F 0 "#PWR0103" H 9400 4200 50  0001 C CNN
 F 1 "+3V3" H 9415 4523 50  0000 C CNN
 F 2 "" H 9400 4350 50  0001 C CNN
@@
 Connection ~ 9700 4350
 Connection ~ 9700 4950
+Text GLabel 8450 1500 0    39   Input ~ 0
+U1_GPIO0
+$Comp
+L power:GND #PWR046
+U 1 1 5EAF6562
+P 8750 2000
+F 0 "#PWR046" H 8750 1750 50  0001 C CNN
+F 1 "GND" H 8755 1827 50  0000 C CNN
+F 2 "" H 8750 2000 50  0001 C CNN
+F 3 "" H 8750 2000 50  0001 C CNN
+	1    8750 2000
+	1    0    0    -1
+$EndComp
+$Comp
+L power:+3V3 #PWR045
+U 1 1 5EB09053
+P 8750 1150
+F 0 "#PWR045" H 8750 1000 50  0001 C CNN
+F 1 "+3V3" H 8750 1300 50  0000 C CNN
+F 2 "" H 8750 1150 50  0001 C CNN
+F 3 "" H 8750 1150 50  0001 C CNN
+	1    8750 1150
+	1    0    0    -1
+$EndComp
+$Comp
+L Device:R R14
+U 1 1 5EB2F921
+P 8750 1300
+F 0 "R14" H 8900 1250 50  0000 C CNN
+F 1 "10k" H 8900 1350 50  0000 C CNN
+F 2 "Resistor_THT:R_Axial_DIN0204_L3.6mm_D1.6mm_P5.08mm_Horizontal" V 8680 1300 50  0001 C CNN
+F 3 "~" H 8750 1300 50  0001 C CNN
+	1    8750 1300
+	-1   0    0    1
+$EndComp
+Wire Wire Line
+	8750 1550 8750 1500
+Wire Wire Line
+	8450 1600 8450 1500
+Wire Wire Line
+	8450 1500 8750 1500
+Connection ~ 8750 1500
+Wire Wire Line
+	8750 1500 8750 1450
+Wire Wire Line
+	8450 1950 8450 1900
+Wire Wire Line
+	8750 1950 8450 1950
+Wire Wire Line
+	8750 2000 8750 1950
+$Comp
+L Device:C C10
+U 1 1 5F64C379
+P 8450 1750
+F 0 "C10" H 8700 1700 50  0000 R CNN
+F 1 "0.1uF" H 8750 1800 50  0000 R CNN
+F 2 "Capacitor_SMD:C_1206_3216Metric_Pad1.42x1.75mm_HandSolder" H 8488 1600 50  0001 C CNN
+F 3 "~" H 8450 1750 50  0001 C CNN
+	1    8450 1750
+	-1   0    0    1
+$EndComp
+$Comp
+L Switch:SW_Push SW6
+U 1 1 5FD62E8D
+P 9700 1750
+F 0 "SW6" V 9750 1500 50  0000 L CNN
+F 1 "RESET" V 9650 1450 50  0000 L CNN
+F 2 "Project_libraries:SW_Push_1P1T_NO_6x6mm_H5mm" H 9700 1950 50  0001 C CNN
+F 3 "~" H 9700 1950 50  0001 C CNN
+	1    9700 1750
+	0    -1   -1   0
+$EndComp
+$Comp
+L Connector:Screw_Terminal_01x02 J1
+U 1 1 5F6B3CD7
+P 900 1100
+F 0 "J1" H 900 800 50  0000 C CNN
+F 1 "PWR 5V" H 900 900 50  0000 C CNN
+F 2 "Project_libraries:PHOENIX_1935161" H 900 1100 50  0001 C CNN
+F 3 "~" H 900 1100 50  0001 C CNN
+	1    900  1100
+	-1   0    0    1
+$EndComp
+$Comp
+L Switch:SW_Push SW5
+U 1 1 5F641C24
+P 8750 1750
+F 0 "SW5" V 8800 1500 50  0000 L CNN
+F 1 "BOOT" V 8700 1600 50  0000 C CNN
+F 2 "Project_libraries:SW_Push_1P1T_NO_6x6mm_H5mm" H 8750 1950 50  0001 C CNN
+F 3 "~" H 8750 1950 50  0001 C CNN
+	1    8750 1750
+	0    -1   -1   0
+$EndComp
+Wire Wire Line
+	10650 1800 10650 1950
+Connection ~ 10650 1950
+Wire Wire Line
+	10650 1500 10650 1700
 $EndSCHEMATC

Commit message: Traced tracks
Connections:
- net GND: now also J9.2 (Pin_2); no longer J9.1 (Pin_1)
- net U2_GPIO2: now also J9.1 (Pin_1); no longer J9.2 (Pin_2)
Changed lines of the file:
@@
-$EndComp
-$Comp
-L Connector:Screw_Terminal_01x02 J9
-U 1 1 5FE3CC4F
-P 10850 1800
-F 0 "J9" H 10800 1500 50  0000 L CNN
-F 1 "LAMP" H 10750 1600 50  0000 L CNN
-F 2 "Project_libraries:PHOENIX_1935161" H 10850 2000 50  0001 C CNN
-F 3 "~" H 10850 2000 50  0001 C CNN
-	1    10850 1800
-	1    0    0    1
 $EndComp
 $Comp
@@
 Wire Wire Line
 	10650 1500 10650 1700
+$Comp
+L Connector:Screw_Terminal_01x02 J9
+U 1 1 5FE3CC4F
+P 10850 1700
+F 0 "J9" H 10800 1900 50  0000 L CNN
+F 1 "LAMP" H 10750 1800 50  0000 L CNN
+F 2 "Project_libraries:PHOENIX_1935161" H 10850 1900 50  0001 C CNN
+F 3 "~" H 10850 1900 50  0001 C CNN
+	1    10850 1700
+	1    0    0    -1
+$EndComp
 $EndSCHEMATC
